File: MCU Datalogger.kicad_sch (KiCad schematic)
At the start: 25 parts, among them U1 24LC1025, U2 24LC1025, U3 DS1337S_, U4 ATMEGA328P-AU, Y1 32.768 KHz, Y2 16 MHz

Commit message: fix the bugs in the schematic.
Connections:
- net SCK: no longer R3.2, U1.6 (SCL), U2.6 (SCL), U3.6 (SCL), U4.28 (PC5)
- net ABC123: no longer names the net of C4.1, U4.20 (AREF)
- new net SCL: R3.2, U1.6 (SCL), U2.6 (SCL), U3.6 (SCL), U4.28 (PC5)
Other:
- sheet Connectors ports: added SCL; removed none
Changed lines of the file:
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@@
 	(wire
 		(pts
-			(xy 242.57 34.29) (xy 242.57 39.37)
-		)
-		(stroke
-			(width 0)
-			(type default)
-		)
-	)
-	(wire
-		(pts
 			(xy 196.85 64.77) (xy 187.96 64.77)
 		)
@@
 		)
 	)
-	(label "abcd"
-		(at 187.96 46.99 0)
-		(effects
-			(font
-				(size 1.27 1.27)
-			)
-			(justify left bottom)
-		)
-	)
 	(label "D3"
 		(at 227.33 54.61 0)
@@
 		)
 	)
-	(label "SCK"
-		(at 173.99 130.81 180)
-		(effects
-			(font
-				(size 1.27 1.27)
-			)
-			(justify right bottom)
-		)
-	)
 	(label "RX"
 		(at 227.33 46.99 0)
@@
 		)
 	)
-	(label "ABC123"
-		(at 228.6 74.93 0)
-		(effects
-			(font
-				(size 1.27 1.27)
-			)
-			(justify left bottom)
-		)
-	)
 	(label "RESET"
 		(at 173.99 154.94 180)
@@
 	)
 	(label "TX"
-		(at 173.99 138.43 180)
+		(at 173.99 135.89 180)
 		(effects
 			(font
@@
 		)
 	)
-	(label "SCK"
-		(at 104.14 147.32 0)
-		(effects
-			(font
-				(size 1.27 1.27)
-			)
-			(justify left bottom)
-		)
-	)
 	(label "Vcc"
 		(at 40.64 149.86 180)
@@
 	)
 	(label "RX"
-		(at 173.99 140.97 180)
+		(at 173.99 138.43 180)
 		(effects
 			(font
@@
 		)
 	)
+	(label "SCL"
+		(at 60.96 147.32 0)
+		(effects
+			(font
+				(size 1.27 1.27)
+			)
+			(justify left bottom)
+		)
+	)
+	(label "SCL"
+		(at 114.3 158.75 0)
+		(effects
+			(font
+				(size 1.27 1.27)
+			)
+			(justify left bottom)
+		)
+	)
 	(label "Vcc"
 		(at 50.8 132.08 0)
@@
 		)
 	)
+	(label "SCL"
+		(at 39.37 46.99 180)
+		(effects
+			(font
+				(size 1.27 1.27)
+			)
+			(justify right bottom)
+		)
+	)
+	(label "SCL"
+		(at 104.14 147.32 0)
+		(effects
+			(font
+				(size 1.27 1.27)
+			)
+			(justify left bottom)
+		)
+	)
 	(label "D7"
 		(at 227.33 64.77 0)
@@
 		)
 	)
-	(label "SCK"
-		(at 114.3 158.75 0)
-		(effects
-			(font
-				(size 1.27 1.27)
-			)
-			(justify left bottom)
-		)
-	)
 	(label "MOSI"
 		(at 173.99 147.32 180)
@@
 		)
 	)
-	(label "SCK"
-		(at 39.37 46.99 180)
+	(label "SCL"
+		(at 173.99 130.81 180)
 		(effects
 			(font
@@
 		)
 	)
-	(label "SCK"
+	(label "SCL"
 		(at 196.85 82.55 180)
 		(effects
@@
 		)
 	)
-	(label "SCK"
-		(at 60.96 147.32 0)
-		(effects
-			(font
-				(size 1.27 1.27)
-			)
-			(justify left bottom)
-		)
-	)
 	(label "D7"
 		(at 203.2 147.32 0)
@@
 		)
 	)
+	(label "SCK"
+		(at 173.99 142.24 180)
+		(effects
+			(font
+				(size 1.27 1.27)
+			)
+			(justify right bottom)
+		)
+	)
 	(symbol
 		(lib_id "DS1337S_:DS1337S_")
@@
 	)
 	(symbol
-		(lib_id "power:PWR_FLAG")
-		(at 242.57 34.29 0)
-		(unit 1)
-		(exclude_from_sim no)
-		(in_bom yes)
-		(on_board yes)
-		(dnp no)
-		(fields_autoplaced yes)
-		(property "Reference" "#FLG01"
-			(at 242.57 32.385 0)
-			(effects
-				(font
-					(size 1.27 1.27)
-				)
-				(hide yes)
-			)
-		)
-		(property "Value" "PWR_FLAG"
-			(at 242.57 29.21 0)
-			(effects
-				(font
-					(size 1.27 1.27)
-				)
-			)
-		)
-		(property "Footprint" ""
-			(at 242.57 34.29 0)
-			(effects
-				(font
-					(size 1.27 1.27)
-				)
-				(hide yes)
-			)
-		)
-		(property "Datasheet" "~"
-			(at 242.57 34.29 0)
-			(effects
-				(font
-					(size 1.27 1.27)
-				)
-				(hide yes)
-			)
-		)
-		(property "Description" "Special symbol for telling ERC where power comes from"
-			(at 242.57 34.29 0)
-			(effects
-				(font
-					(size 1.27 1.27)
-				)
-				(hide yes)
-			)
-		)
-		(pin "1"
-		)
-		(instances
-			(project ""
-				(path "/b34ba724-37f1-4069-92d1-dfc9c20970e0"
-					(reference "#FLG01")
-					(unit 1)
-				)
-			)
-		)
-	)
-	(symbol
 		(lib_id "Device:R")
 		(at 125.73 152.4 0)
@@
 		)
 		(pin "TX" output
-			(at 173.99 138.43 180)
+			(at 173.99 135.89 180)
 			(effects
 				(font
@@
 			)
 		)
-		(pin "SCK" passive
-			(at 173.99 130.81 180)
-			(effects
-				(font
-					(size 1.27 1.27)
-				)
-				(justify left)
-			)
-		)
 		(pin "SDA" bidirectional
 			(at 173.99 128.27 180)
@@
 		)
 		(pin "RX" input
-			(at 173.99 140.97 180)
+			(at 173.99 138.43 180)
 			(effects
 				(font
@@
 			)
 		)
+		(pin "SCK" passive
+			(at 173.99 142.24 180)
+			(effects
+				(font
+					(size 1.27 1.27)
+				)
+				(justify left)
+			)
+		)
+		(pin "SCL" passive
+			(at 173.99 130.81 180)
+			(effects
+				(font
+					(size 1.27 1.27)
+				)
+				(justify left)
+			)
+		)
